File: inputSwitchboard/connectors.kicad_sch (KiCad schematic)
At the start: 0 parts

Commit message: finished schematic
Parts:
- added J3: INPUT SEL, TerminalBlock_Phoenix:TerminalBlock_Phoenix_MKDS-1,5-3-5.08_1x03_P5.08mm_Horizontal, symbol Connector:Screw_Terminal_01x03
- added J4: OUTPUT SEL, TerminalBlock_Phoenix:TerminalBlock_Phoenix_MKDS-1,5-3-5.08_1x03_P5.08mm_Horizontal, symbol Connector:Screw_Terminal_01x03
- added J5, J6, J7: Screw_Terminal_01x07, symbol Connector:Screw_Terminal_01x07
- added J8: Screw_Terminal_01x14, symbol Connector:Screw_Terminal_01x14
- added J9: Screw_Terminal_01x04, symbol Connector:Screw_Terminal_01x04
- added R5, R6, R7, R8: 4k7R, Resistor_SMD:R_0603_1608Metric, symbol Device:R
Connections:
- new net +3V3: J3.1 (Pin_1), J4.1 (Pin_1)
- new net CTRL-EXT-1-CLK: J6.2 (Pin_2)
- new net CTRL-EXT-2-LATCH: J6.3 (Pin_3)
- new net CTRL-EXT-3-D1: J6.4 (Pin_4)
- new net CTRL-EXT-4-VCC: J6.5 (Pin_5)
- new net CTRL-EXT-5-D3: J6.6 (Pin_6)
- new net CTRL-EXT-6-D4: J6.7 (Pin_7)
- new net CTRL-INT-1-CLK: J5.2 (Pin_2)
- new net CTRL-INT-2-LATCH: J5.3 (Pin_3)
- new net CTRL-INT-3-D1: J5.4 (Pin_4)
- new net CTRL-INT-4-VCC: J5.5 (Pin_5)
- new net CTRL-INT-5-D3: J5.6 (Pin_6)
- new net CTRL-INT-6-D4: J5.7 (Pin_7)
- new net GND: J5.1 (Pin_1), J6.1 (Pin_1), J7.1 (Pin_1), R5.2, R6.2, R7.2, R8.2
- new net GPIO10: J8.10 (Pin_10)
- new net GPIO11: J8.9 (Pin_9)
- new net GPIO12: J8.8 (Pin_8)
- new net GPIO13: J8.7 (Pin_7)
- new net GPIO14: J8.6 (Pin_6)
- new net GPIO15: J8.5 (Pin_5)
- new net GPIO16: J8.4 (Pin_4)
- new net GPIO17: J8.3 (Pin_3)
- new net GPIO18: J8.2 (Pin_2)
- new net GPIO19: J8.1 (Pin_1)
- new net GPIO26-ADC0: J9.4 (Pin_4)
- new net GPIO27-ADC1: J9.3 (Pin_3)
- new net GPIO28-ADC2: J9.2 (Pin_2)
- new net GPIO29-ADC3: J9.1 (Pin_1)
- new net GPIO6: J8.14 (Pin_14)
- new net GPIO7: J8.13 (Pin_13)
- new net GPIO8: J8.12 (Pin_12)
- new net GPIO9: J8.11 (Pin_11)
- new net INPUT-SEL-NC: J3.3 (Pin_3), R8.1
- new net INPUT-SEL-NO: J3.2 (Pin_2), R7.1
- new net OUTPUT-SEL-NC: J4.3 (Pin_3), R5.1
- new net OUTPUT-SEL-NO: J4.2 (Pin_2), R6.1
- new net PROC-NES-1-CLK: J7.2 (Pin_2)
- new net PROC-NES-2-LATCH: J7.3 (Pin_3)
- new net PROC-NES-3-D1: J7.4 (Pin_4)
- new net PROC-NES-4-VCC: J7.5 (Pin_5)
- new net PROC-NES-5-D3: J7.6 (Pin_6)
- new net PROC-NES-6-D4: J7.7 (Pin_7)
Other:
- note added: "exposed GPIO for expansion TODO: Add silkscreen labels"
- note removed: "daughterboard"

Commit message: Proofread, started to route
Parts:
- J5: value Screw_Terminal_01x07 -> INT CTRL; footprint (none) -> TerminalBlock:TerminalBlock_MaiXu_MX126-5.0-07P_1x07_P5.00mm; now not fitted; now left out of the parts list
- J6: value Screw_Terminal_01x07 -> EXT CTRL; footprint (none) -> TerminalBlock:TerminalBlock_MaiXu_MX126-5.0-07P_1x07_P5.00mm; now not fitted; now left out of the parts list
- J7: value Screw_Terminal_01x07 -> NES; footprint (none) -> TerminalBlock:TerminalBlock_MaiXu_MX126-5.0-07P_1x07_P5.00mm; now not fitted; now left out of the parts list
- J8: value Screw_Terminal_01x14 -> GPIO; footprint (none) -> TerminalBlock:TerminalBlock_MaiXu_MX126-5.0-14P_1x14_P5.00mm; now left out of the parts list
- J9: value Screw_Terminal_01x04 -> GPIO-ADC; footprint (none) -> TerminalBlock:TerminalBlock_MaiXu_MX126-5.0-04P_1x04_P5.00mm; now left out of the parts list
Changed lines of the file:
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@@
 		(unit 1)
 		(exclude_from_sim no)
-		(in_bom yes)
+		(in_bom no)
 		(on_board yes)
 		(dnp yes)
@@
 			)
 		)
-		(property "Value" "Screw_Terminal_01x04"
+		(property "Value" "GPIO-ADC"
 			(at 193.04 123.1899 0)
 			(effects
@@
 			)
 		)
-		(property "Footprint" ""
+		(property "Footprint" "TerminalBlock:TerminalBlock_MaiXu_MX126-5.0-04P_1x04_P5.00mm"
 			(at 190.5 120.65 0)
 			(effects
@@
 		(unit 1)
 		(exclude_from_sim no)
-		(in_bom yes)
+		(in_bom no)
 		(on_board yes)
 		(dnp yes)
@@
 			)
 		)
-		(property "Value" "Screw_Terminal_01x14"
+		(property "Value" "GPIO"
 			(at 245.11 120.6499 0)
 			(effects
@@
 			)
 		)
-		(property "Footprint" ""
+		(property "Footprint" "TerminalBlock:TerminalBlock_MaiXu_MX126-5.0-14P_1x14_P5.00mm"
 			(at 242.57 118.11 0)
 			(effects
@@
 		(unit 1)
 		(exclude_from_sim no)
-		(in_bom yes)
-		(on_board yes)
-		(dnp no)
+		(in_bom no)
+		(on_board yes)
+		(dnp yes)
 		(fields_autoplaced yes)
 		(property "Reference" "J7"
@@
 			)
 		)
-		(property "Value" "Screw_Terminal_01x07"
+		(property "Value" "NES"
 			(at 245.11 81.2799 0)
 			(effects
@@
 			)
 		)
-		(property "Footprint" ""
+		(property "Footprint" "TerminalBlock:TerminalBlock_MaiXu_MX126-5.0-07P_1x07_P5.00mm"
 			(at 242.57 80.01 0)
 			(effects
@@
 		(unit 1)
 		(exclude_from_sim no)
-		(in_bom yes)
-		(on_board yes)
-		(dnp no)
+		(in_bom no)
+		(on_board yes)
+		(dnp yes)
 		(fields_autoplaced yes)
 		(property "Reference" "J5"
@@
 			)
 		)
-		(property "Value" "Screw_Terminal_01x07"
+		(property "Value" "INT CTRL"
 			(at 80.01 81.2799 0)
 			(effects
@@
 			)
 		)
-		(property "Footprint" ""
+		(property "Footprint" "TerminalBlock:TerminalBlock_MaiXu_MX126-5.0-07P_1x07_P5.00mm"
 			(at 77.47 80.01 0)
 			(effects
@@
 		(unit 1)
 		(exclude_from_sim no)
-		(in_bom yes)
-		(on_board yes)
-		(dnp no)
+		(in_bom no)
+		(on_board yes)
+		(dnp yes)
 		(fields_autoplaced yes)
 		(property "Reference" "J6"
@@
 			)
 		)
-		(property "Value" "Screw_Terminal_01x07"
+		(property "Value" "EXT CTRL"
 			(at 160.02 81.2799 0)
 			(effects
@@
 			)
 		)
-		(property "Footprint" ""
+		(property "Footprint" "TerminalBlock:TerminalBlock_MaiXu_MX126-5.0-07P_1x07_P5.00mm"
 			(at 157.48 80.01 0)
 			(effects

Commit message: finished routing
Parts:
- removed J9: GPIO-ADC, TerminalBlock:TerminalBlock_MaiXu_MX126-5.0-04P_1x04_P5.00mm, symbol Connector:Screw_Terminal_01x04
Changed lines of the file:
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@@
-	(wire
-		(pts
-			(xy 185.42 120.65) (xy 182.88 120.65)
-		)
-		(stroke
-			(width 0)
-			(type default)
-		)
-	)
 	(wire
 		(pts
@@
 	(wire
 		(pts
-			(xy 185.42 123.19) (xy 182.88 123.19)
-		)
-		(stroke
-			(width 0)
-			(type default)
-		)
-	)
-	(wire
-		(pts
 			(xy 149.86 62.23) (xy 157.48 62.23)
 		)
@@
 	(wire
 		(pts
-			(xy 185.42 118.11) (xy 182.88 118.11)
-		)
-		(stroke
-			(width 0)
-			(type default)
-		)
-	)
-	(wire
-		(pts
 			(xy 234.95 77.47) (xy 237.49 77.47)
 		)
@@
 		(pts
 			(xy 69.85 62.23) (xy 77.47 62.23)
-		)
-		(stroke
-			(width 0)
-			(type default)
-		)
-	)
-	(wire
-		(pts
-			(xy 185.42 125.73) (xy 182.88 125.73)
 		)
 		(stroke
@@
 		)
 	)
-	(global_label "GPIO29-ADC3"
-		(shape bidirectional)
-		(at 182.88 118.11 180)
-		(fields_autoplaced yes)
-		(effects
-			(font
-				(size 1.27 1.27)
-			)
-			(justify right)
-		)
-		(property "Intersheetrefs" "${INTERSHEET_REFS}"
-			(at 165.4787 118.11 0)
-			(effects
-				(font
-					(size 1.27 1.27)
-				)
-				(justify right)
-				(hide yes)
-			)
-		)
-	)
 	(global_label "GPIO15"
 		(shape bidirectional)
@@
 		)
 	)
-	(global_label "GPIO26-ADC0"
-		(shape bidirectional)
-		(at 182.88 125.73 180)
-		(fields_autoplaced yes)
-		(effects
-			(font
-				(size 1.27 1.27)
-			)
-			(justify right)
-		)
-		(property "Intersheetrefs" "${INTERSHEET_REFS}"
-			(at 165.4787 125.73 0)
-			(effects
-				(font
-					(size 1.27 1.27)
-				)
-				(justify right)
-				(hide yes)
-			)
-		)
-	)
 	(global_label "CTRL-INT-5-D3"
 		(shape output)
@@
 		)
 	)
-	(global_label "GPIO28-ADC2"
-		(shape bidirectional)
-		(at 182.88 120.65 180)
-		(fields_autoplaced yes)
-		(effects
-			(font
-				(size 1.27 1.27)
-			)
-			(justify right)
-		)
-		(property "Intersheetrefs" "${INTERSHEET_REFS}"
-			(at 165.4787 120.65 0)
-			(effects
-				(font
-					(size 1.27 1.27)
-				)
-				(justify right)
-				(hide yes)
-			)
-		)
-	)
 	(global_label "PROC-NES-4-VCC"
 		(shape input)
@@
 		(property "Intersheetrefs" "${INTERSHEET_REFS}"
 			(at 130.6068 85.09 0)
-			(effects
-				(font
-					(size 1.27 1.27)
-				)
-				(justify right)
-				(hide yes)
-			)
-		)
-	)
-	(global_label "GPIO27-ADC1"
-		(shape bidirectional)
-		(at 182.88 123.19 180)
-		(fields_autoplaced yes)
-		(effects
-			(font
-				(size 1.27 1.27)
-			)
-			(justify right)
-		)
-		(property "Intersheetrefs" "${INTERSHEET_REFS}"
-			(at 165.4787 123.19 0)
 			(effects
 				(font
@@
 					(unit 1)
 				)
-			)
-		)
-	)
-	(symbol
-		(lib_id "Connector:Screw_Terminal_01x04")
-		(at 190.5 120.65 0)
-		(unit 1)
-		(exclude_from_sim no)
-		(in_bom no)
-		(on_board yes)
-		(dnp yes)
-		(fields_autoplaced yes)
-		(property "Reference" "J9"
-			(at 193.04 120.6499 0)
-			(effects
-				(font
-					(size 1.27 1.27)
-				)
-				(justify left)
-			)
-		)
-		(property "Value" "GPIO-ADC"
-			(at 193.04 123.1899 0)
-			(effects
-				(font
-					(size 1.27 1.27)
-				)
-				(justify left)
-			)
-		)
-		(property "Footprint" "TerminalBlock:TerminalBlock_MaiXu_MX126-5.0-04P_1x04_P5.00mm"
-			(at 190.5 120.65 0)
-			(effects
-				(font
-					(size 1.27 1.27)
-				)
-				(hide yes)
-			)
-		)
-		(property "Datasheet" "~"
-			(at 190.5 120.65 0)
-			(effects
-				(font
-					(size 1.27 1.27)
-				)
-				(hide yes)
-			)
-		)
-		(property "Description" "Generic screw terminal, single row, 01x04, script generated (kicad-library-utils/schlib/autogen/connector/)"
-			(at 190.5 120.65 0)
-			(effects
-				(font
-					(size 1.27 1.27)
-				)
-				(hide yes)
-			)
-		)
-		(pin "3"
-		)
-		(pin "2"
-		)
-		(pin "4"
-		)
-		(pin "1"
-		)
-		(instances
-			(project ""
-				(path "/45e54069-11e8-4323-b4ab-97e83e8fb66c/8d754924-1ee4-41b7-afda-6e43d02b1969"
-					(reference "J9")
-					(unit 1)
-				)

Commit message: fixed more stuff and polished routing
Parts:
- removed J8: GPIO, TerminalBlock:TerminalBlock_MaiXu_MX126-5.0-14P_1x14_P5.00mm, symbol Connector:Screw_Terminal_01x14
- J3, J4: now not fitted; now left out of the parts list
Other:
- note removed: "exposed GPIO for expansion TODO: Add silkscreen labels"
