File: inputSwitchboard/inputSwitchboard.kicad_pcb (KiCad board)
At the start: 2 copper layers, 66 parts, among them J1 DATA, J10 BOOTSEL, J11 RESET, J12 DEBUG, J2 POWER, J3 INPUT SEL, J4 OUTPUT SEL, J5 INT CTRL, J6 EXT CTRL, J7 NES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

Commit message: finished routing
Parts:
- removed J9: GPIO-ADC, TerminalBlock:TerminalBlock_MaiXu_MX126-5.0-04P_1x04_P5.00mm
- moved C18 110.4 mm to (95.8, 51.2)
- moved Y1 99.7 mm to (92.9, 57.9), turned to 90 degrees
- moved R14 93.5 mm to (95.5, 54.1)
- moved C1 89.5 mm to (75.6, 99.6)
- moved C2 89.5 mm to (75.6, 101.3)
- moved C3 64.9 mm to (91.2, 92.7)
- moved C4 64.9 mm to (91.2, 94.5)
- moved D1 58.2 mm to (112.1, 106.7)
- moved R4 53.8 mm to (110.1, 103.2), turned to 90 degrees
- moved D2 51.9 mm to (106.8, 106.7)
- moved R9 34.1 mm to (106.8, 103.2), turned to 90 degrees
- moved C11 28.5 mm to (121.3, 122.5)
- moved C12 28.5 mm to (121.3, 124.2)
- moved C13 28.5 mm to (121.3, 126.0)
- moved C15 28.5 mm to (126.3, 122.7)
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Connections:
- J1 pad Sh1: (no net) -> GND
- J2 pad Sh1: (no net) -> GND
Routing:
- net PROC-NES-4-VCC: track 0.00 -> 165.2 mm, vias 0 -> 4
- net PROC-NES-3-D1: track 0.00 -> 155.9 mm, vias 0 -> 3
- net PROC-NES-1-CLK: track 0.00 -> 136.1 mm, vias 0 -> 4
- net PROC-NES-2-LATCH: track 0.00 -> 100.2 mm, vias 0 -> 4
- net +5V: track 176.9 -> 214.7 mm, vias 12 -> 13
- net GND: track 92.4 -> 129.0 mm, vias 28 -> 37
- net Net-(J10-Pin_2): track 6.56 -> 40.3 mm
- net Net-(U2-GPIO25): track 0.00 -> 29.5 mm, vias 0 -> 2
- net XOUT: track 0.00 -> 23.6 mm, vias 0 -> 2
- net NAND-SD0: track 8.88 -> 32.4 mm, vias 0 -> 2
- net USBD-: track 56.5 -> 33.8 mm, vias 2 -> 0
- net USBD+: track 59.1 -> 37.4 mm, vias 0 -> 2
- net NAND-SCLK: track 11.7 -> 32.8 mm, vias 0 -> 2
- net +3V3: track 40.0 -> 60.6 mm, vias 4 -> 12
- net NAND-SD3: track 13.2 -> 33.5 mm, vias 0 -> 2
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
Commit message: fixed more stuff and polished routing
Parts:
- removed J8: GPIO, TerminalBlock:TerminalBlock_MaiXu_MX126-5.0-14P_1x14_P5.00mm
- added ?: , , F.Cu at (140.3, 39.3)
- added ?: , , F.Cu at (74.8, 39.3)
- added G***: LOGO, imports:rickroll, F.Cu at (93.8, 74.5)
- D1, D2: footprint LED_SMD:LED_0201_0603Metric -> LED_SMD:LED_0603_1608Metric
- moved C17 63.5 mm to (94.6, 71.2), turned to 90 degrees
- moved C15 53.5 mm to (104.6, 73.8)
- moved C13 52.5 mm to (104.9, 76.1)
- moved C12 52.4 mm to (104.6, 74.6)
- moved C16 50.9 mm to (117.6, 74.3), turned to -90 degrees
- moved C11 48.2 mm to (103.5, 77.7), turned to -90 degrees
- moved R12 32.5 mm to (117.4, 61.2)
- moved R13 32.5 mm to (115.8, 61.2)
- moved U10 26.8 mm to (114.3, 70.3)
- moved R14 20.2 mm to (92.6, 74.0)
- moved C18 17.8 mm to (92.4, 68.7)
- moved J11 14.9 mm to (107.9, 83.8)
- moved C2 14.2 mm to (88.2, 94.8), turned to -90 degrees
- moved Y1 13.3 mm to (92.4, 71.2), turned to 180 degrees
- moved C1 11.3 mm to (86.8, 101.6), turned to 90 degrees
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Routing:
- net +3V3: track 60.6 -> 217.7 mm
- net PROC-NES-4-VCC: track 165.2 -> 80.2 mm, vias 4 -> 1
- net CTRL-EXT-4-VCC: track 78.1 -> 13.1 mm, vias 2 -> 1
- net Net-(J12-Pin_2): track 0.00 -> 42.0 mm, vias 0 -> 2
- net Net-(J12-Pin_1): track 0.00 -> 41.3 mm, vias 0 -> 2
- net Net-(J10-Pin_2): track 40.3 -> 6.36 mm
- net XOUT: track 23.6 -> 2.14 mm, vias 2 -> 0
- net NAND-SD0: track 32.4 -> 12.3 mm, vias 2 -> 0
- net NAND-SCLK: track 32.8 -> 14.0 mm, vias 2 -> 0
- net NAND-SD3: track 33.5 -> 15.0 mm, vias 2 -> 0
- net GND: track 129.0 -> 111.7 mm, vias 37 -> 155
- net RUN: track 44.1 -> 29.2 mm
- net PROC-NES-1-CLK: track 136.1 -> 149.7 mm, vias 4 -> 6
- net XIN: track 16.6 -> 4.52 mm, vias 2 -> 0
- net NAND-SD2: track 26.3 -> 15.3 mm, vias 2 -> 0
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- added copper zone on F.Cu, net GND
- removed copper zone on F.Cu, net +3V3
Other:
- board outline added: 95 x 85 mm
- board text added: "2025 @cybdo with support from Hack Club Blueprint made with <3"
- board text added: "NES Controller Multiplexer (Switchboard) v1"
- board text added: "PWR"
- board text added: "STATUS"

Commit message: done!
Parts:
- removed ? (x2): , 
- added H3: MountingHole, MountingHole:MountingHole_4.3mm_M4, F.Cu at (74.8, 39.3)
- added H4: MountingHole, MountingHole:MountingHole_4.3mm_M4, F.Cu at (140.3, 39.3)
- U3, U4, U5, U6, U7, U8: footprint Package_SO:MSOP-10-1EP_3x3mm_P0.5mm_EP1.68x1.88mm -> Package_SO:VSSOP-10_3x3mm_P0.5mm
- moved R15 1.44 mm to (112.4, 79.2)
- moved R10 0.92 mm to (105.5, 81.3)
- moved R11 0.92 mm to (103.6, 81.3)
Connections:
- U2 pad 11: GPIO8 -> unconnected-(U2-GPIO8-Pad11)
- U2 pad 12: GPIO9 -> unconnected-(U2-GPIO9-Pad12)
- U2 pad 13: GPIO10 -> unconnected-(U2-GPIO10-Pad13)
- U2 pad 14: GPIO11 -> unconnected-(U2-GPIO11-Pad14)
- U2 pad 15: GPIO12 -> unconnected-(U2-GPIO12-Pad15)
- U2 pad 16: GPIO13 -> unconnected-(U2-GPIO13-Pad16)
- U2 pad 17: GPIO14 -> unconnected-(U2-GPIO14-Pad17)
- U2 pad 18: GPIO15 -> unconnected-(U2-GPIO15-Pad18)
- U2 pad 27: GPIO16 -> unconnected-(U2-GPIO16-Pad27)
- U2 pad 28: GPIO17 -> unconnected-(U2-GPIO17-Pad28)
- U2 pad 29: GPIO18 -> unconnected-(U2-GPIO18-Pad29)
- U2 pad 30: GPIO19 -> unconnected-(U2-GPIO19-Pad30)
- U2 pad 38: GPIO26-ADC0 -> unconnected-(U2-GPIO26_ADC0-Pad38)
- U2 pad 39: GPIO27-ADC1 -> unconnected-(U2-GPIO27_ADC1-Pad39)
- U2 pad 40: GPIO28-ADC2 -> unconnected-(U2-GPIO28_ADC2-Pad40)
- U2 pad 41: GPIO29-ADC3 -> unconnected-(U2-GPIO29_ADC3-Pad41)
- U2 pad 8: GPIO6 -> unconnected-(U2-GPIO6-Pad8)
- U2 pad 9: GPIO7 -> unconnected-(U2-GPIO7-Pad9)
Routing:
- net +3V3: track 217.7 -> 207.4 mm
- net PROC-RP-5-D3: track 40.7 -> 33.8 mm
- net GND: track 111.7 -> 108.5 mm, vias 155 -> 171
- net IN-SEL: track 62.2 -> 60.0 mm
- net Net-(U5-D-): track 9.24 -> 11.2 mm
- net +5V: track 204.8 -> 206.7 mm
- net CTRL-EXT-1-CLK: track 48.8 -> 48.0 mm
- net RUN: track 29.2 -> 30.0 mm
- net OUT-SEL: track 47.9 -> 47.2 mm
