File: inputSwitchboard/inputSwitchboard.kicad_sch (KiCad schematic)
At the start: 22 parts, among them J1 DATA, J2 POWER, J3-INPUT-SEL Conn_01x03_Socket, J4-OUTPUT-SEL Conn_01x03_Socket, U1 AMS1117-3.3, U3 TS3USB30EDGSR, U4 TS3USB30EDGSR, U5 TS3USB30EDGSR, U6 TS3USB30EDGSR, U7 TS3USB30EDGSR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

Commit message: finished schematic
Parts:
- removed J3-INPUT-SEL, J4-OUTPUT-SEL: Conn_01x03_Socket, Connector_PinHeader_1.00mm:PinHeader_1x03_P1.00mm_Vertical, symbol Connector:Conn_01x03_Socket
- removed R5, R6, R7, R8: 4k7R, Resistor_SMD:R_0603_1608Metric, symbol Device:R
- D1: value PWR -> PWR_LED
Connections:
- net +5V: no longer U6.2 (D1+)
- new net PROC-NES-4-VCC: U6.2 (D1+)
Other:
- moved on the sheet: J2

Commit message: Proofread, started to route
Parts:
- added H1, H2: MountingHole, MountingHole:MountingHole_4.3mm_M4, symbol Mechanical:MountingHole
- added R16, R17: 4k7R, Resistor_SMD:R_0603_1608Metric, symbol Device:R
- added R18, R19: 6k8R, Resistor_SMD:R_0603_1608Metric, symbol Device:R
- added U11, U12: ~, Package_TO_SOT_SMD:SOT-23-5, symbol New_Library:SY6280AAC
- J1, J2: footprint (none) -> imports:TYPE-C-31-M-12
- U3, U4, U5, U6, U7, U8: value TS3USB30EDGSR -> CH442E; footprint Package_SO:VSSOP-10_3x3mm_P0.5mm -> Package_SO:MSOP-10-1EP_3x3mm_P0.5mm_EP1.68x1.88mm
Connections:
- net +3V3: now also U5.2 (D1+), U5.3 (D2+); no longer U3.10 (VCC), U4.10 (VCC), U5.10 (VCC), U6.10 (VCC), U7.10 (VCC), U8.10 (VCC)
- net +5V: now also U3.10 (VCC), U4.10 (VCC), U5.10 (VCC), U6.10 (VCC), U7.10 (VCC), U8.10 (VCC), U11.5 (IN); no longer U6.3 (D2+)
- net CTRL-EXT-4-VCC: now also U11.1 (OUT); no longer U5.2 (D1+)
- net CTRL-INT-4-VCC: now also U12.1 (OUT); no longer U5.3 (D2+)
- net GND: now also R16.2, R17.2, R18.2, R19.2, U11.2 (GND), U12.2 (GND)
- net PROC-NES-4-VCC: now also U12.5 (IN); no longer U6.2 (D1+)
- new net: R18.1, U11.3 (ISET)
- new net: R19.1, U12.3 (ISET)
- new net NES-VCC-TOGGLE: R17.1, U12.4 (EN), U6.2 (D1+)
- new net RP-VCC-TOGGLE: R16.1, U11.4 (EN), U6.3 (D2+)
Other:
- moved on the sheet: U7, U8

Commit message: fixed more stuff and polished routing
Parts:
- added H3, H4: MountingHole, MountingHole:MountingHole_4.3mm_M4, symbol Mechanical:MountingHole
Changed lines of the file:
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@@
+	)
+	(symbol
+		(lib_id "Mechanical:MountingHole")
+		(at 81.28 194.31 0)
+		(unit 1)
+		(exclude_from_sim no)
+		(in_bom no)
+		(on_board yes)
+		(dnp no)
+		(fields_autoplaced yes)
+		(property "Reference" "H3"
+			(at 83.82 193.0399 0)
+			(effects
+				(font
+					(size 1.27 1.27)
+				)
+				(justify left)
+			)
+		)
+		(property "Value" "MountingHole"
+			(at 83.82 195.5799 0)
+			(effects
+				(font
+					(size 1.27 1.27)
+				)
+				(justify left)
+			)
+		)
+		(property "Footprint" "MountingHole:MountingHole_4.3mm_M4"
+			(at 81.28 194.31 0)
+			(effects
+				(font
+					(size 1.27 1.27)
+				)
+				(hide yes)
+			)
+		)
+		(property "Datasheet" "~"
+			(at 81.28 194.31 0)
+			(effects
+				(font
+					(size 1.27 1.27)
+				)
+				(hide yes)
+			)
+		)
+		(property "Description" "Mounting Hole without connection"
+			(at 81.28 194.31 0)
+			(effects
+				(font
+					(size 1.27 1.27)
+				)
+				(hide yes)
+			)
+		)
+		(instances
+			(project "inputSwitchboard"
+				(path "/45e54069-11e8-4323-b4ab-97e83e8fb66c"
+					(reference "H3")
+					(unit 1)
+				)
+			)
+		)
 	)
 	(symbol
@@
 					(unit 1)
 				)
+			)
+		)
+	)
+	(symbol
+		(lib_id "Mechanical:MountingHole")
+		(at 121.92 190.5 0)
+		(unit 1)
+		(exclude_from_sim no)
+		(in_bom no)
+		(on_board yes)
+		(dnp no)
+		(fields_autoplaced yes)
+		(property "Reference" "H4"
+			(at 124.46 189.2299 0)
+			(effects
+				(font
+					(size 1.27 1.27)
+				)
+				(justify left)
+			)
+		)
+		(property "Value" "MountingHole"
+			(at 124.46 191.7699 0)
+			(effects
+				(font
+					(size 1.27 1.27)
+				)
+				(justify left)
+			)
+		)
+		(property "Footprint" "MountingHole:MountingHole_4.3mm_M4"
+			(at 121.92 190.5 0)
+			(effects
+				(font
+					(size 1.27 1.27)
+				)
+				(hide yes)
+			)
+		)
+		(property "Datasheet" "~"
+			(at 121.92 190.5 0)
+			(effects
+				(font
+					(size 1.27 1.27)
+				)
+				(hide yes)
+			)
+		)
+		(property "Description" "Mounting Hole without connection"
+			(at 121.92 190.5 0)
+			(effects
+				(font
+					(size 1.27 1.27)
+				)
+				(hide yes)
+			)
+		)
+		(instances
+			(project "inputSwitchboard"
+				(path "/45e54069-11e8-4323-b4ab-97e83e8fb66c"
+					(reference "H4")
+					(unit 1)
+				)

Commit message: done!
Parts:
- D1: footprint LED_SMD:LED_0201_0603Metric -> LED_SMD:LED_0603_1608Metric
- U3, U4, U5, U6, U7, U8: footprint Package_SO:MSOP-10-1EP_3x3mm_P0.5mm_EP1.68x1.88mm -> Package_SO:VSSOP-10_3x3mm_P0.5mm
Connections:
- net GND: now also J1.Sh1 (SHIELD), J2.Sh1 (SHIELD); no longer J1.S1 (SHIELD), J2.S1 (SHIELD)
Changed lines of the file:
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@@
 	)
 	(symbol
-		(lib_name "SY6280AAC_1")
 		(lib_id "New_Library:SY6280AAC")
 		(at 160.02 120.65 0)
@@
 			)
 		)
-		(property "Footprint" "Package_SO:MSOP-10-1EP_3x3mm_P0.5mm_EP1.68x1.88mm"
+		(property "Footprint" "Package_SO:VSSOP-10_3x3mm_P0.5mm"
 			(at 34.29 152.4 0)
 			(effects
@@
 			)
 		)
-		(property "Footprint" "LED_SMD:LED_0201_0603Metric"
+		(property "Footprint" "LED_SMD:LED_0603_1608Metric"
 			(at 156.21 38.1 0)
 			(effects
@@
 			)
 		)
-		(property "Footprint" "Package_SO:MSOP-10-1EP_3x3mm_P0.5mm_EP1.68x1.88mm"
+		(property "Footprint" "Package_SO:VSSOP-10_3x3mm_P0.5mm"
 			(at 34.29 99.06 0)
 			(effects
@@
 		(on_board yes)
 		(dnp no)
-		(fields_autoplaced yes)
 		(property "Reference" "U4"
 			(at 107.5533 95.25 0)
@@
 			)
 		)
-		(property "Footprint" "Package_SO:MSOP-10-1EP_3x3mm_P0.5mm_EP1.68x1.88mm"
+		(property "Footprint" "Package_SO:VSSOP-10_3x3mm_P0.5mm"
 			(at 125.73 116.84 0)
 			(effects
@@
 			)
 		)
-		(property "Footprint" "Package_SO:MSOP-10-1EP_3x3mm_P0.5mm_EP1.68x1.88mm"
+		(property "Footprint" "Package_SO:VSSOP-10_3x3mm_P0.5mm"
 			(at 125.73 170.18 0)
 			(effects
@@
 			)
 		)
-		(pin "S1"
+		(pin "Sh1"
 		)
 		(pin "B7"
@@
 		(on_board yes)
 		(dnp no)
-		(fields_autoplaced yes)
 		(property "Reference" "U7"
 			(at 194.8881 74.93 0)
@@
 			)
 		)
-		(property "Footprint" "Package_SO:MSOP-10-1EP_3x3mm_P0.5mm_EP1.68x1.88mm"
+		(property "Footprint" "Package_SO:VSSOP-10_3x3mm_P0.5mm"
 			(at 171.45 78.74 0)
 			(effects
@@
 			)
 		)
-		(property "Footprint" "Package_SO:MSOP-10-1EP_3x3mm_P0.5mm_EP1.68x1.88mm"
+		(property "Footprint" "Package_SO:VSSOP-10_3x3mm_P0.5mm"
 			(at 262.89 96.52 0)
 			(effects
@@
 			)
 		)
-		(pin "S1"
+		(pin "Sh1"
 		)
 		(pin "B7"
