File: inputSwitchboard/rp2040.kicad_sch (KiCad schematic)
At the start: 6 parts, among them U2 RP2040, U9 TXS0108EPW

Commit message: finished schematic
Parts:
- added C10, C11, C12, C14, C15, C16, C6, C7, C8, C9: 100nF, Capacitor_SMD:C_0201_0603Metric, symbol Device:C
- added C13, C5: 1uF, Capacitor_SMD:C_0201_0603Metric, symbol Device:C
- added C17, C18: 15pF, Capacitor_SMD:C_0201_0603Metric, symbol Device:C
- added J10: Conn_01x03_Pin, Connector:FanPinHeader_1x03_P2.54mm_Vertical, symbol Connector:Conn_01x03_Pin
- added R10, R11: 5k1R, Resistor_SMD:R_0603_1608Metric, symbol Device:R
- added R12, R14: 1kR, Resistor_SMD:R_0603_1608Metric, symbol Device:R
- added R13: 10kR, Resistor_SMD:R_0603_1608Metric, symbol Device:R
- added U10: W25Q128JVS, Package_SO:SOIC-8_5.3x5.3mm_P1.27mm, symbol Memory_Flash:W25Q128JVS
- added Y1: ABM8-272-T3, ABM8-272-T3:XTAL_ABM8-272-T3, symbol ABM8-272-T3:ABM8-272-T3
Connections:
- net +3V3: now also C10.1, C11.1, C12.1, C16.1, C5.1, C6.1, C7.1, C8.1, C9.1, R13.2, U10.8 (VCC)
- net GND: now also U2.1 (IOVDD), U2.10 (IOVDD), U2.22 (IOVDD), U2.33 (IOVDD), U2.42 (IOVDD), U2.43 (ADC_AVDD), U2.44 (VREG_IN), U2.48 (USB_VDD), U2.49 (IOVDD), C10.2, C11.2, C12.2, C13.2, C14.2, C15.2, C16.2, C18.2, C5.2, C6.2, C7.2, C8.2, C9.2, J10.3 (Pin_3), U10.4 (GND), Y1.2 (GND), Y1.4 (GND)
- net GPIO8: now reaches U2.11 (GPIO8)
- net GPIO9: now reaches U2.12 (GPIO9)
- net GPIO10: now reaches U2.13 (GPIO10)
- net GPIO11: now reaches U2.14 (GPIO11)
- net GPIO12: now reaches U2.15 (GPIO12)
- net GPIO13: now reaches U2.16 (GPIO13)
- net GPIO14: now reaches U2.17 (GPIO14)
- net GPIO15: now reaches U2.18 (GPIO15)
- net XIN: now reaches U2.20 (XIN)
- net XIN: now also C17.1, Y1.1
- net XOUT: now reaches U2.21 (XOUT)
- net XOUT: now also R14.2
- net +1V1: now reaches U2.23 (DVDD), U2.50 (DVDD)
- net +1V1: now also U2.45 (VREG_VOUT), C13.1, C14.1, C15.1
- net GPIO16: now reaches U2.27 (GPIO16)
- net GPIO17: now reaches U2.28 (GPIO17)
- net GPIO18: now reaches U2.29 (GPIO18)
- net GPIO19: now reaches U2.30 (GPIO19)
- net GPIO26-ADC0: now reaches U2.38 (GPIO26_ADC0)
- net GPIO27-ADC1: now reaches U2.39 (GPIO27_ADC1)
- net GPIO28-ADC2: now reaches U2.40 (GPIO28_ADC2)
- net GPIO29-ADC3: now reaches U2.41 (GPIO29_ADC3)
- net at U2.46 (USB_DM): now also R11.2
- net at U2.47 (USB_DP): now also R10.2
- net NAND-SD3: now reaches U2.51 (QSPI_SD3)
- net NAND-SD3: now also U10.7 (~{HOLD}/~{RESET}/IO_{3})
- net NAND-SCLK: now reaches U2.52 (QSPI_SCLK)
- net NAND-SCLK: now also U10.6 (CLK)
- net NAND-SD0: now reaches U2.53 (QSPI_SD0)
- net NAND-SD0: now also U10.5 (DI/IO_{0})
- net NAND-SD2: now reaches U2.54 (QSPI_SD2)
- net NAND-SD2: now also U10.3 (~{WP}/IO_{2})
- net NAND-SD1: now reaches U2.55 (QSPI_SD1)
- net NAND-SD1: now also U10.2 (DO/IO_{1})
- net NAND-SS: now reaches U2.56 (QSPI_SS)
- net NAND-SS: now also R12.2, R13.1, U10.1 (~{CS})
- net GPIO6: now reaches U2.8 (GPIO6)
- net GPIO7: now reaches U2.9 (GPIO7)
- new net: J10.2 (Pin_2), R12.1
- new net: C18.1, R14.1, Y1.3
- new net USBD+: R10.1
- new net USBD-: R11.1
- no-connect marks 6 -> 7
Other:
- note added: "c13 next to 45, c14, c15 next to 23, 50"
- note added: "c5 next to 44, c6-12 next to 1, 10, 22, 33, 42, 43, (48,49)"
- moved on the sheet: C3, C4, D2, R9, U9

Commit message: Proofread, started to route
Parts:
- added J11: RESET, Connector:FanPinHeader_1x03_P2.54mm_Vertical, symbol Connector:Conn_01x03_Pin
- added J12: DEBUG, Connector:FanPinHeader_1x03_P2.54mm_Vertical, symbol Connector:Conn_01x03_Pin
- added R15: 4k7R, Resistor_SMD:R_0603_1608Metric, symbol Device:R
- J10: value Conn_01x03_Pin -> BOOTSEL; now not fitted; now left out of the parts list
- Y1: footprint ABM8-272-T3:XTAL_ABM8-272-T3 -> imports:XTAL_ABM8-272-T3
Connections:
- net +3V3: now also U2.1 (IOVDD), U2.10 (IOVDD), U2.22 (IOVDD), U2.33 (IOVDD), U2.42 (IOVDD), U2.43 (ADC_AVDD), U2.44 (VREG_IN), U2.48 (USB_VDD), U2.49 (IOVDD), R15.2
- net GND: now also C17.2, U2.19 (TESTEN), J11.3 (Pin_3), J12.3 (Pin_3); no longer U2.1 (IOVDD), U2.10 (IOVDD), U2.22 (IOVDD), U2.33 (IOVDD), U2.42 (IOVDD), U2.43 (ADC_AVDD), U2.44 (VREG_IN), U2.48 (USB_VDD), U2.49 (IOVDD)
- net at U2.24 (SWCLK): now also J12.1 (Pin_1)
- net at U2.25 (SWD): now also J12.2 (Pin_2)
- net RUN: now reaches U2.26 (RUN)
- net RUN: now also J11.2 (Pin_2), R15.1
- no-connect marks 7 -> 8

Commit message: finished routing
Connections:
- net GPIO26-ADC0: no longer names the net of U2.38 (GPIO26_ADC0)
- net GPIO27-ADC1: no longer names the net of U2.39 (GPIO27_ADC1)
- net GPIO28-ADC2: no longer names the net of U2.40 (GPIO28_ADC2)
- net GPIO29-ADC3: no longer names the net of U2.41 (GPIO29_ADC3)
- no-connect marks 8 -> 12
Changed lines of the file:
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@@
+	)
+	(no_connect
+		(at 109.22 118.11)
 	)
 	(no_connect
@@
 	)
 	(no_connect
+		(at 109.22 113.03)
+	)
+	(no_connect
 		(at 160.02 87.63)
 	)
@@
 	)
 	(no_connect
+		(at 109.22 115.57)
+	)
+	(no_connect
 		(at 180.34 87.63)
 	)
+	(no_connect
+		(at 109.22 110.49)
+	)
 	(wire
 		(pts
@@
 	(wire
 		(pts
-			(xy 111.76 113.03) (xy 109.22 113.03)
-		)
-		(stroke
-			(width 0)
-			(type default)
-		)
-	)
-	(wire
-		(pts
 			(xy 109.22 85.09) (xy 114.3 85.09)
 		)
@@
 	(wire
 		(pts
-			(xy 111.76 110.49) (xy 109.22 110.49)
-		)
-		(stroke
-			(width 0)
-			(type default)
-		)
-	)
-	(wire
-		(pts
 			(xy 109.22 137.16) (xy 109.22 142.24)
 		)
@@
 	(wire
 		(pts
-			(xy 111.76 115.57) (xy 109.22 115.57)
-		)
-		(stroke
-			(width 0)
-			(type default)
-		)
-	)
-	(wire
-		(pts
 			(xy 163.83 138.43) (xy 163.83 146.05)
 		)
@@
 		(pts
 			(xy 195.58 156.21) (xy 195.58 157.48)
-		)
-		(stroke
-			(width 0)
-			(type default)
-		)
-	)
-	(wire
-		(pts
-			(xy 111.76 118.11) (xy 109.22 118.11)
 		)
 		(stroke
@@
 		)
 	)
-	(global_label "GPIO29-ADC3"
-		(shape bidirectional)
-		(at 111.76 118.11 0)
-		(fields_autoplaced yes)
-		(effects
-			(font
-				(size 1.27 1.27)
-			)
-			(justify left)
-		)
-		(property "Intersheetrefs" "${INTERSHEET_REFS}"
-			(at 129.1613 118.11 0)
-			(effects
-				(font
-					(size 1.27 1.27)
-				)
-				(justify left)
-				(hide yes)
-			)
-		)
-	)
-	(global_label "GPIO26-ADC0"
-		(shape bidirectional)
-		(at 111.76 110.49 0)
-		(fields_autoplaced yes)
-		(effects
-			(font
-				(size 1.27 1.27)
-			)
-			(justify left)
-		)
-		(property "Intersheetrefs" "${INTERSHEET_REFS}"
-			(at 129.1613 110.49 0)
-			(effects
-				(font
-					(size 1.27 1.27)
-				)
-				(justify left)
-				(hide yes)
-			)
-		)
-	)
 	(global_label "GPIO14"
 		(shape bidirectional)
@@
 		)
 	)
-	(global_label "GPIO27-ADC1"
-		(shape bidirectional)
-		(at 111.76 113.03 0)
-		(fields_autoplaced yes)
-		(effects
-			(font
-				(size 1.27 1.27)
-			)
-			(justify left)
-		)
-		(property "Intersheetrefs" "${INTERSHEET_REFS}"
-			(at 129.1613 113.03 0)
-			(effects
-				(font
-					(size 1.27 1.27)
-				)
-				(justify left)
-				(hide yes)
-			)
-		)
-	)
 	(global_label "NAND-SCLK"
 		(shape output)
@@
 				(hide yes)
 			)
-		)
-	)
-	(global_label "GPIO28-ADC2"
-		(shape bidirectional)
-		(at 111.76 115.57 0)
-		(fields_autoplaced yes)
-		(effects
-			(font
-				(size 1.27 1.27)
-			)
-			(justify left)
-		)
-		(property "Intersheetrefs" "${INTERSHEET_REFS}"
-			(at 129.1613 115.57 0)
-			(effects
-				(font
-					(size 1.27 1.27)
-				)
-				(justify left)
-				(hide yes)
-			)

Commit message: fixed more stuff and polished routing
Connections:
- net GPIO10: no longer names the net of U2.13 (GPIO10)
- net GPIO11: no longer names the net of U2.14 (GPIO11)
- net GPIO12: no longer names the net of U2.15 (GPIO12)
- net GPIO13: no longer names the net of U2.16 (GPIO13)
- net GPIO14: no longer names the net of U2.17 (GPIO14)
- net GPIO15: no longer names the net of U2.18 (GPIO15)
- net GPIO16: no longer names the net of U2.27 (GPIO16)
- net GPIO17: no longer names the net of U2.28 (GPIO17)
- net GPIO18: no longer names the net of U2.29 (GPIO18)
- net GPIO19: no longer names the net of U2.30 (GPIO19)
- net GPIO6: no longer names the net of U2.8 (GPIO6)
- net GPIO7: no longer names the net of U2.9 (GPIO7)
- net GPIO8: no longer names the net of U2.11 (GPIO8)
- net GPIO9: no longer names the net of U2.12 (GPIO9)
- no-connect marks 12 -> 26

Commit message: done!
Parts:
- D2: footprint LED_SMD:LED_0201_0603Metric -> LED_SMD:LED_0603_1608Metric
- Y1: footprint imports:XTAL_ABM8-272-T3 -> ABM8-272-T3:XTAL_ABM8-272-T3
Changed lines of the file:
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@@
 			)
 		)
-		(property "Footprint" "LED_SMD:LED_0201_0603Metric"
+		(property "Footprint" "LED_SMD:LED_0603_1608Metric"
 			(at 153.67 120.65 0)
 			(effects
@@
 			)
 		)
-		(property "Footprint" "imports:XTAL_ABM8-272-T3"
+		(property "Footprint" "ABM8-272-T3:XTAL_ABM8-272-T3"
 			(at 179.07 146.05 0)
 			(effects
